Commit message: update s2 model

File: limo_s2/limo_s2_description/urdf/limo_s2.xacro (robot description, xacro)
@@ -26,5 +26,5 @@
             <origin xyz="0.095 0 -0.035" rpy="0 0 1.57" />
             <geometry>
-                <mesh filename="package://limo_s2_description/meshes/dae/base_link.dae" scale="1 1 1"/>
+                <mesh filename="package://limo_s2_description/meshes/dae/base_link_2.dae" scale="0.001 0.001 0.001"/>
             </geometry>
         </visual>

File: limo_s2/limo_s2_description/urdf/limo_xacro.xacro (robot description, xacro)
@@ -11,5 +11,5 @@
                 <origin xyz="0.01 -0.064 0.064" rpy="0 0 -1.57" />
                 <geometry>
-                    <mesh filename="package://limo_s2_description/meshes/dae/LIMO_S2_mailun_1.dae" />
+                    <mesh filename="package://limo_s2_description/meshes/dae/mailun_1.dae" />
                 </geometry>
             </visual>
@@ -38,5 +38,5 @@
                 <origin xyz="0 0 0" rpy="0 0 0" />
                 <geometry>
-                    <mesh filename="package://limo_s2_description/meshes/dae/LIMO_S2_mailun_2.dae" />
+                    <mesh filename="package://limo_s2_description/meshes/dae/mailun_2.dae" />
                 </geometry>
             </visual>
@@ -72,5 +72,5 @@
                     <mesh filename="package://limo_s2_description/meshes/laser_Link.STL" />
                 </geometry>
-                <material name='laser_material'>
+                <material name=''>
                     <ambient>0.1 0.1 0.1 1</ambient>
                     <diffuse>0.1 0.1 0.2 1</diffuse>
@@ -110,7 +110,7 @@
                 <origin xyz="0.21 0 -0.13" rpy="0 0 1.57 "/>
                 <geometry>
-                    <mesh filename="package://limo_s2_description/meshes/dae/camera_Link.dae" />
+                    <mesh filename="package://limo_s2_description/meshes/dae/camera.dae" />
                 </geometry>
-                <material name='depth_camera_material'>
+                <material name=''>
                     <ambient>0.1 0.1 0.1 1</ambient>
                     <diffuse>0.1 0.1 0.2 1</diffuse>
@@ -158,5 +158,5 @@
                     <box size="0.001 0.001 0.001"/>
                 </geometry>
-                <material name='imu_material'>
+                <material name=''>
                     <ambient>0.1 0.1 0.1 1</ambient>
                     <diffuse>0.1 0.1 0.2 1</diffuse>
