Commit message: update hunter se

File: hunter_se/hunter_se_description/urdf/hunter_se_description.urdf (robot description, URDF)
Before this commit: robot hunter_se_description, 9 links, 8 joints
Links:
- link base_link: mass 0.01 -> 10
- link fr_left_link: mass 0.01 -> 1
- link fr_right_link: mass 0.01 -> 1
- link fr_steer_left_link: mass 0.01 -> 1
- link fr_steer_right_link: mass 0.01 -> 1
- link re_left_link: mass 0.01 -> 1
- link re_right_link: mass 0.01 -> 1
