Commit message: add hunter_se ranger_mini sim

File: hunter_se/hunter_se_description/urdf/hunter_se_description_with_box.xacro (robot description, xacro)
@@ -369,3 +369,103 @@
       xyz="0 0 1" />
   </joint>
+  <link
+    name="box_link">
+    <inertial>
+      <origin
+        xyz="0 0 0"
+        rpy="0 0 0" />
+      <mass
+        value="0.01" />
+      <inertia
+        ixx="0.0176011208398464"
+        ixy="-8.00593138518773E-09"
+        ixz="-0.000253357559513648"
+        iyy="0.0175967847225325"
+        iyz="-5.65898177386586E-11"
+        izz="0.0326650290732703" />
+    </inertial>
+    <visual>
+      <origin
+        xyz="0 0 0"
+        rpy="0 0 0" />
+      <geometry>
+        <box size="0.5 0.28 0.2"/>
+      </geometry>
+      <material
+        name="">
+        <color
+          rgba="1 1 1 1" />
+      </material>
+    </visual>
+    <collision>
+      <origin
+        xyz="0 0 0"
+        rpy="0 0 0" />
+      <geometry>
+        <box size="0.5 0.28 0.2"/>
+      </geometry>
+    </collision>
+  </link>
+  <joint
+    name="box_joint"
+    type="fixed">
+    <origin
+      xyz="0.2 0 0.1"
+      rpy="0 0 0" />
+    <parent
+      link="base_link" />
+    <child
+      link="box_link" />
+    <axis
+      xyz="0 0 0" />
+  </joint>
+  <link
+    name="laser_link">
+    <inertial>
+      <origin
+        xyz="0 0 0"
+        rpy="0 0 0" />
+      <mass
+        value="0.01" />
+      <inertia
+        ixx="0.0176011208398464"
+        ixy="-8.00593138518773E-09"
+        ixz="-0.000253357559513648"
+        iyy="0.0175967847225325"
+        iyz="-5.65898177386586E-11"
+        izz="0.0326650290732703" />
+    </inertial>
+    <visual>
+      <origin
+        xyz="0 0 0"
+        rpy="0 0 0" />
+      <geometry>
+      <cylinder radius="0.01" length="0.01"/>
+      </geometry>
+      <material
+        name="">
+        <color
+          rgba="1 1 1 1" />
+      </material>
+    </visual>
+    <collision>
+      <origin
+        xyz="0 0 0"
+        rpy="0 0 0" />
+      <geometry>
+      <cylinder radius="0.01" length="0.01"/>
+      </geometry>
+    </collision>
+  </link>
+  <joint
+    name="laser_joint"
+    type="fixed">
+    <origin
+      xyz="0.43 0 0.2"
+      rpy="0 0 0" />
+    <parent
+      link="base_link" />
+    <child
+      link="laser_link" />
+  </joint>
 </robot>

File: hunter_se/hunter_se_gazebo/xacro/hunter_se_gazebo copy.xacro (robot description, xacro)
@@ -4,5 +4,5 @@
      For more information, please see http://wiki.ros.org/sw_urdf_exporter -->
 <robot
-  name="hunter_se_description">
+  name="hunter_se">
   <link
     name="base_link">
@@ -27,5 +27,5 @@
       <geometry>
         <mesh
-          filename="package://hunter_se_description/meshes/base_link.STL" />
+          filename="file://$(find hunter_se_description)/meshes/base_link.STL" />
       </geometry>
       <material
@@ -41,5 +41,5 @@
       <geometry>
         <mesh
-          filename="package://hunter_se_description/meshes/base_link.STL" />
+          filename="file://$(find hunter_se_description)/meshes/base_link.STL" />
       </geometry>
     </collision>
@@ -84,5 +84,5 @@
   </link>
   <joint
-    name="fr_steer_left_jiont"
+    name="fr_steer_left_joint"
     type="revolute">
     <origin
@@ -123,5 +123,5 @@
       <geometry>
         <mesh
-          filename="package://hunter_se_description/meshes/fr_left_link.STL" />
+          filename="file://$(find hunter_se_description)/meshes/fr_left_link.STL" />
       </geometry>
       <material
@@ -137,5 +137,5 @@
       <geometry>
         <mesh
-          filename="package://hunter_se_description/meshes/fr_left_link.STL" />
+          filename="file://$(find hunter_se_description)/meshes/fr_left_link.STL" />
       </geometry>
     </collision>
@@ -193,5 +193,5 @@
   </link>
   <joint
-    name="fr_steer_right_link"
+    name="fr_steer_right_joint"
     type="revolute">
     <origin
@@ -232,5 +232,5 @@
       <geometry>
         <mesh
-          filename="package://hunter_se_description/meshes/fr_right_link.STL" />
+          filename="file://$(find hunter_se_description)/meshes/fr_right_link.STL" />
       </geometry>
       <material
@@ -246,5 +246,5 @@
       <geometry>
         <mesh
-          filename="package://hunter_se_description/meshes/fr_right_link.STL" />
+          filename="file://$(find hunter_se_description)/meshes/fr_right_link.STL" />
       </geometry>
     </collision>
@@ -285,5 +285,5 @@
       <geometry>
         <mesh
-          filename="package://hunter_se_description/meshes/re_left_link.STL" />
+          filename="file://$(find hunter_se_description)/meshes/re_left_link.STL" />
       </geometry>
       <material
@@ -299,10 +299,10 @@
       <geometry>
         <mesh
-          filename="package://hunter_se_description/meshes/re_left_link.STL" />
-      </geometry>
-    </collision>
-  </link>
-  <joint
-    name="re_left_jiont"
+          filename="file://$(find hunter_se_description)/meshes/re_left_link.STL" />
+      </geometry>
+    </collision>
+  </link>
+  <joint
+    name="re_left_joint"
     type="continuous">
     <origin
@@ -338,5 +338,5 @@
       <geometry>
         <mesh
-          filename="package://hunter_se_description/meshes/re_right_link.STL" />
+          filename="file://$(find hunter_se_description)/meshes/re_right_link.STL" />
       </geometry>
       <material
@@ -352,10 +352,10 @@
       <geometry>
         <mesh
-          filename="package://hunter_se_description/meshes/re_right_link.STL" />
-      </geometry>
-    </collision>
-  </link>
-  <joint
-    name="re_right_jiont"
+          filename="file://$(find hunter_se_description)/meshes/re_right_link.STL" />
+      </geometry>
+    </collision>
+  </link>
+  <joint
+    name="re_right_joint"
     type="continuous">
     <origin
@@ -369,3 +369,81 @@
       xyz="0 0 1" />
   </joint>
+   <link name="steering_wheel_link">
+        <inertial>
+            <origin xyz="0.0 0.0 0.0" rpy="0.0 0.0 0.0"/>
+            <mass value="1"/>
+            <inertia ixx="0.01" ixy="0.0" ixz="0.0" iyy="0.01" iyz="0.0" izz="0.01"/>
+        </inertial>
+        <visual>
+            <origin xyz="-0.23 -0.194 0.1" rpy="1.57 0 3.14 " />
+            <geometry>
+                <cylinder radius="0.001" length="0.001"/>
+            </geometry>
+        </visual>
+        <collision>
+            <origin xyz="0 0 0.008" rpy="0 0 0" />
+            <geometry>
+                <cylinder radius="0.001" length="0.001"/>
+            </geometry>
+        </collision>
+    </link>
+    <joint name="steering_whee_joint" type="revolute">
+        <origin xyz="-0.23 0.206 -0.1" rpy="0 0 0" />
+        <parent link="base_link"/>
+        <child link="steering_wheel_link"/>
+        <axis xyz="0 0 1" rpy="0 0 0" />
+        <limit effort="5" velocity="6.28"  lower="-2.1" upper="2.1" />
+    </joint>
+     <gazebo>
+            <plugin name="ackermann_controller" filename="libgazebo_ros_ackermann_drive.so">
+                <update_rate>100</update_rate>
+                <front_left_joint>fr_left_joint</front_left_joint>
+                <front_right_joint>fr_right_joint</front_right_joint>
+                <rear_left_joint>re_left_joint</rear_left_joint>
+                <rear_right_joint>re_right_joint</rear_right_joint>
+                <left_steering_joint>fr_steer_left_joint</left_steering_joint>
+                <right_steering_joint>fr_steer_right_joint</right_steering_joint>
+                <steering_wheel_joint>steering_whee_joint</steering_wheel_joint>
+                <left_steering_pid_gain>10000 100 10</left_steering_pid_gain>
+                <left_steering_i_rang>0 0</left_steering_i_rang>
+                <right_steering_pid_gain>10000 100 10</right_steering_pid_gain>
+                <right_steering_i_rang>0 0</right_steering_i_rang>
+                <linear_velocity_pid_gain>0.5 10 0.001</linear_velocity_pid_gain>
+                <linear_velocity_i_range>0 0</linear_velocity_i_range>
+                <max_steer>0.523598767</max_steer>
+                <wheel_separation>0.172</wheel_separation>
+                <wheel_diameter>0.09</wheel_diameter>
+                <max_wheel_torque>20</max_wheel_torque>
+                <max_wheel_acceleration>1.0</max_wheel_acceleration>
+                <command_topic>cmd_vel</command_topic>
+                <publish_odom>true</publish_odom>
+                <publish_odom_tf>true</publish_odom_tf>
+                <publish_wheel_tf>true</publish_wheel_tf>
+                <odometry_topic>odom</odometry_topic>
+                <odometry_frame>odom</odometry_frame>
+                <robot_base_frame>base_link</robot_base_frame>
+            </plugin>
+        </gazebo>
+<gazebo>
+    <plugin name="gazebo_ros_control" filename="libgazebo_ros_control.so" />
+</gazebo>
+<!--
+<gazebo>
+    <plugin name="object_controller" filename="libgazebo_ros_planar_move.so">
+      <ros>
+        <namespace>/demo</namespace>
+        <remapping>cmd_vel:=custom_cmd_vel</remapping>
+        <remapping>odom:=custom_odom</remapping>
+      </ros>
+      <update_rate>100</update_rate>
+      <publish_rate>10</publish_rate>
+      <publish_odom>true</publish_odom>
+      <publish_odom_tf>true</publish_odom_tf>
+      <odometry_frame>odom_demo</odometry_frame>
+      <robot_base_frame>base_link</robot_base_frame>
+      <covariance_x>0.0001</covariance_x>
+      <covariance_y>0.0001</covariance_y>
+      <covariance_yaw>0.01</covariance_yaw>
+    </plugin>
+</gazebo> -->
 </robot>
