Commit message: modify autokit.urdf

File: autokit/urdf/autokit.urdf (robot description, URDF)
Before this commit: robot autokit, 2 links, 1 joints
Links:
- link box_Link: geometry collision mesh filename=package://autokit/meshes/box_Link.STL; visual mesh filename=package://autokit/meshes/box_Link.STL
