Commit message: complete hunter

File: hunter/hunter2_base/urdf/hunter2_base_gazebo.xacro (robot description, xacro)
@@ -12,5 +12,5 @@
         rpy="0 0 0" />
       <mass
-        value="1.02945169536679" />
+        value="21.02945169536679" />
       <inertia
         ixx="0.0332370959804736"
@@ -52,5 +52,5 @@
         rpy="0 0 0" />
       <mass
-        value="0.8526" />
+        value="7.8526" />
       <inertia
         ixx="0.063827"
@@ -108,5 +108,5 @@
         rpy="0 0 0" />
       <mass
-        value="0.7007" />
+        value="7.7007" />
       <inertia
         ixx="0.063724"
@@ -153,4 +153,5 @@
     <axis
       xyz="0 0 -1" />
+      <dynamics damping="0.0" friction="3"/>
   </joint>
   <link
@@ -161,5 +162,5 @@
         rpy="0 0 0" />
       <mass
-        value="0.696" />
+        value="7.696" />
       <inertia
         ixx="0.063704"
@@ -217,5 +218,5 @@
         rpy="0 0 0" />
       <mass
-        value="0.5613" />
+        value="7.5613" />
       <inertia
         ixx="0.063626"
@@ -262,4 +263,5 @@
     <axis
       xyz="0 0 -1" />
+      <dynamics damping="0.0" friction="3"/>
   </joint>
   <link
@@ -270,5 +272,5 @@
         rpy="0 0 0" />
       <mass
-        value="0.6692" />
+        value="7.6692" />
       <inertia
         ixx="0.063699"
@@ -315,9 +317,5 @@
     <axis
       xyz="0 0 -1" />
-    <limit
-      lower="-3.14"
-      upper="3.14"
-      effort="0"
-      velocity="0" />
+     <dynamics damping="0.0" friction="3"/>
   </joint>
   <link
@@ -328,5 +326,5 @@
         rpy="0 0 0" />
       <mass
-        value="0.7133" />
+        value="7.7133" />
       <inertia
         ixx="0.06373"
@@ -373,9 +371,5 @@
     <axis
       xyz="0 0 -1" />
-    <limit
-      lower="-3.14"
-      upper="3.14"
-      effort="0"
-      velocity="0" />
+     <dynamics damping="0.0" friction="3"/>
   </joint>
   <link
@@ -485,15 +479,44 @@
     <axis
       xyz="0 0 1" />
+    <dynamics damping="0.0" friction="3"/>
   </joint>
   <gazebo reference="front_left_wheel_link">
+    <mu1>0.9</mu1>
+    <mu2>0.9</mu2>
+    <kp>500000.0</kp>
+    <kd>10.0</kd>
+    <minDepth>0.001</minDepth>
+    <maxVel>0.1</maxVel>
+    <fdir1>1 0 0</fdir1>
       <material>Gazebo/Grey </material>
       </gazebo>
   <gazebo reference="front_right_wheel_link">
+      <mu1>0.9</mu1>
+    <mu2>0.9</mu2>
+    <kp>500000.0</kp>
+    <kd>10.0</kd>
+    <minDepth>0.001</minDepth>
+    <maxVel>0.1</maxVel>
+    <fdir1>1 0 0</fdir1>
       <material>Gazebo/Grey </material>
       </gazebo>
   <gazebo reference="right_rear_link">
+      <mu1>0.9</mu1>
+    <mu2>0.9</mu2>
+    <kp>500000.0</kp>
+    <kd>10.0</kd>
+    <minDepth>0.001</minDepth>
+    <maxVel>0.1</maxVel>
+    <fdir1>1 0 0</fdir1>
       <material>Gazebo/Grey </material>
       </gazebo>
   <gazebo reference="left_rear_link">
+      <mu1>0.9</mu1>
+    <mu2>0.9</mu2>
+    <kp>500000.0</kp>
+    <kd>10.0</kd>
+    <minDepth>0.001</minDepth>
+    <maxVel>0.1</maxVel>
+    <fdir1>1 0 0</fdir1>
       <material>Gazebo/Grey </material>
       </gazebo>

Commit message: complete hunter really

File: hunter/hunter2_base/urdf/hunter2_base_gazebo.xacro (robot description, xacro)
@@ -153,5 +153,5 @@
     <axis
       xyz="0 0 -1" />
-      <dynamics damping="0.0" friction="3"/>
+      <dynamics damping="0.0" friction="2"/>
   </joint>
   <link
@@ -263,5 +263,5 @@
     <axis
       xyz="0 0 -1" />
-      <dynamics damping="0.0" friction="3"/>
+      <dynamics damping="0.0" friction="2"/>
   </joint>
   <link
@@ -317,5 +317,5 @@
     <axis
       xyz="0 0 -1" />
-     <dynamics damping="0.0" friction="3"/>
+     <dynamics damping="0.0" friction="2"/>
   </joint>
   <link
@@ -371,5 +371,5 @@
     <axis
       xyz="0 0 -1" />
-     <dynamics damping="0.0" friction="3"/>
+     <dynamics damping="0.0" friction="2"/>
   </joint>
   <link
@@ -479,9 +479,9 @@
     <axis
       xyz="0 0 1" />
-    <dynamics damping="0.0" friction="3"/>
+    <dynamics damping="0.0" friction="2"/>
   </joint>
   <gazebo reference="front_left_wheel_link">
-    <mu1>0.9</mu1>
-    <mu2>0.9</mu2>
+    <mu1>0.8</mu1>
+    <mu2>0.8</mu2>
     <kp>500000.0</kp>
     <kd>10.0</kd>
@@ -492,6 +492,6 @@
       </gazebo>
   <gazebo reference="front_right_wheel_link">
-      <mu1>0.9</mu1>
-    <mu2>0.9</mu2>
+      <mu1>0.8</mu1>
+    <mu2>0.8</mu2>
     <kp>500000.0</kp>
     <kd>10.0</kd>
@@ -502,6 +502,6 @@
       </gazebo>
   <gazebo reference="right_rear_link">
-      <mu1>0.9</mu1>
-    <mu2>0.9</mu2>
+      <mu1>0.8</mu1>
+    <mu2>10</mu2>
     <kp>500000.0</kp>
     <kd>10.0</kd>
@@ -512,6 +512,6 @@
       </gazebo>
   <gazebo reference="left_rear_link">
-      <mu1>0.9</mu1>
-    <mu2>0.9</mu2>
+      <mu1>0.8</mu1>
+    <mu2>10</mu2>
     <kp>500000.0</kp>
     <kd>10.0</kd>

Commit message: complete hunter_se

File: hunter/hunter2_base/urdf/hunter2_base_gazebo.xacro (robot description, xacro)
@@ -111,8 +111,8 @@
       <inertia
         ixx="0.063724"
-        ixy="-3.8745E-08"
-        ixz="2.2753E-07"
+        ixy="0"
+        ixz="0"
         iyy="0.063724"
-        iyz="-4.88E-08"
+        iyz="0"
         izz="0.11072" />
     </inertial>
@@ -153,5 +153,5 @@
     <axis
       xyz="0 0 -1" />
-      <dynamics damping="0.0" friction="2"/>
+      <dynamics damping="0.0" friction="15"/>
   </joint>
   <link
@@ -221,8 +221,8 @@
       <inertia
         ixx="0.063626"
-        ixy="-6.4092E-08"
-        ixz="-2.0164E-08"
+        ixy="0"
+        ixz="0"
         iyy="0.063626"
-        iyz="6.4721E-08"
+        iyz="0"
         izz="0.11054" />
     </inertial>
@@ -263,5 +263,5 @@
     <axis
       xyz="0 0 -1" />
-      <dynamics damping="0.0" friction="2"/>
+      <dynamics damping="0.0" friction="15"/>
   </joint>
   <link
@@ -275,8 +275,8 @@
       <inertia
         ixx="0.063699"
-        ixy="-2.542E-07"
-        ixz="2.638E-08"
+        ixy="0"
+        ixz="0"
         iyy="0.063699"
-        iyz="-5.9934E-08"
+        iyz="0"
         izz="0.11067" />
     </inertial>
@@ -317,5 +317,5 @@
     <axis
       xyz="0 0 -1" />
-     <dynamics damping="0.0" friction="2"/>
+     <dynamics damping="0.0" friction="15"/>
   </joint>
   <link
@@ -329,8 +329,8 @@
       <inertia
         ixx="0.06373"
-        ixy="2.5408E-07"
-        ixz="2.6379E-08"
+        ixy="0"
+        ixz="0"
         iyy="0.06373"
-        iyz="5.9941E-08"
+        iyz="0"
         izz="0.11073" />
     </inertial>
@@ -371,5 +371,5 @@
     <axis
       xyz="0 0 -1" />
-     <dynamics damping="0.0" friction="2"/>
+     <dynamics damping="0.0" friction="15"/>
   </joint>
   <link
@@ -479,5 +479,5 @@
     <axis
       xyz="0 0 1" />
-    <dynamics damping="0.0" friction="2"/>
+    <dynamics damping="0.0" friction="15"/>
   </joint>
   <gazebo reference="front_left_wheel_link">

File: hunter_se/hunter_se_description/urdf/hunter_se_description.urdf (robot description, URDF)
Before this commit: robot hunter_se_description, 9 links, 8 joints
Links:
- link base_link: mass 10 -> 24.73
- link fr_left_link: mass 1 -> 3.149
- link fr_right_link: mass 1 -> 3.149
- link fr_steer_left_link: mass 1 -> 3.149
- link fr_steer_right_link: mass 1 -> 3.149
- link re_left_link: mass 1 -> 3.149
- link re_right_link: mass 1 -> 3.149
Joints:
- removed joint re_left_jiont
- removed joint re_right_jiont
- added joint re_left_joint: type continuous, parent base_link, child re_left_link, origin xyz=-0.2078 0.252 -0.158 rpy=1.5708 0 0, axis 0 0 -1
- added joint re_right_joint: type continuous, parent base_link, child re_right_link, origin xyz=-0.2078 -0.252 -0.158 rpy=-1.5708 0 0, axis 0 0 1

Commit message: complete scout2.0

File: hunter/hunter2_base/urdf/hunter2_base_gazebo.xacro (robot description, xacro)
@@ -483,5 +483,5 @@
   <gazebo reference="front_left_wheel_link">
     <mu1>0.8</mu1>
-    <mu2>0.8</mu2>
+    <mu2>10</mu2>
     <kp>500000.0</kp>
     <kd>10.0</kd>
@@ -493,5 +493,5 @@
   <gazebo reference="front_right_wheel_link">
       <mu1>0.8</mu1>
-    <mu2>0.8</mu2>
+    <mu2>10</mu2>
     <kp>500000.0</kp>
     <kd>10.0</kd>

File: scout/scout_description/urdf/scout_v2.xacro (robot description, xacro)
@@ -45,5 +45,5 @@
     <link name="inertial_link">
         <inertial>
-            <mass value="200" />
+            <mass value="50" />
             <!-- <mass value="50" /> -->
             <!-- <origin xyz="-0.00065 -0.085 0.062" />

File: scout/scout_description/urdf/scout_wheel_type1.xacro (robot description, xacro)
@@ -54,4 +54,5 @@
             <xacro:insert_block name="joint_pose"/>
             <axis xyz="0 -1 0" rpy="0 0 0" />
+            <dynamics damping="0.0" friction="20"/>
         </joint>
     </xacro:macro>

File: scout/scout_description/urdf/scout_wheel_type2.xacro (robot description, xacro)
@@ -54,4 +54,5 @@
             <xacro:insert_block name="joint_pose"/>
             <axis xyz="0 -1 0" rpy="0 0 0" />
+            <dynamics damping="0.0" friction="20"/>
         </joint>
     </xacro:macro>
