Commit message: complete ranger mini

File: ranger/ranger_mini/urdf/ranger_mini.gazebo.xacro (robot description, xacro)
@@ -23,36 +23,56 @@
   	<gazebo reference="rear_left_steering_link">
 	  <!-- <selfCollide>false</selfCollide> -->
-      <mu1 value="1.5" />
-      <mu2 value="1.5" />
+      <mu1 value="0.5" />
+      <mu2 value="0.5" />
       <material>Gazebo/Grey</material>
     </gazebo>
   	<gazebo reference="rear_right_steering_link">
 	  <!-- <selfCollide>false</selfCollide> -->
-      <mu1 value="1.5" />
-      <mu2 value="1.5" />
+      <mu1 value="0.5" />
+      <mu2 value="0.5" />
       <material>Gazebo/Grey</material>
     </gazebo>
     <gazebo reference="ffl_wheel_link">
       <!-- <selfCollide>false</selfCollide> -->
-      <mu1 value="10" />
-      <mu2 value="10" />
+      <mu1>0.8</mu1>
+    <mu2>0.8</mu2>
+    <kp>10000000.0</kp>
+    <kd>1.0</kd>
+    <minDepth>0.001</minDepth>
+    <maxVel>0.1</maxVel>
+    <fdir1>1 0 0</fdir1>
       <material>Gazebo/Grey</material>
     </gazebo>
     <gazebo reference="ffr_wheel_link">
       <!-- <selfCollide>false</selfCollide> -->
-      <mu1 value="10" />
-      <mu2 value="10" />
+      <mu1>0.8</mu1>
+    <mu2>0.8</mu2>
+    <kp>10000000.0</kp>
+    <kd>1.0</kd>
+    <minDepth>0.001</minDepth>
+    <maxVel>0.1</maxVel>
+    <fdir1>1 0 0</fdir1>
       <material>Gazebo/Grey</material>
     </gazebo>
     <gazebo reference="rfl_wheel_link">
       <!-- <selfCollide>false</selfCollide> -->
-      <mu1 value="10" />
-      <mu2 value="10" />
+      <mu1>0.8</mu1>
+    <mu2>0.8</mu2>
+    <kp>10000000.0</kp>
+    <kd>1.0</kd>
+    <minDepth>0.001</minDepth>
+    <maxVel>0.1</maxVel>
+    <fdir1>1 0 0</fdir1>
       <material>Gazebo/Grey</material>
     </gazebo>
     <gazebo reference="rfr_wheel_link">
       <!-- <selfCollide>false</selfCollide> -->
-      <mu1 value="10" />
-      <mu2 value="10" />
+      <mu1>0.8</mu1>
+    <mu2>0.8</mu2>
+    <kp>10000000.0</kp>
+    <kd>1.0</kd>
+    <minDepth>0.001</minDepth>
+    <maxVel>0.1</maxVel>
+    <fdir1>1 0 0</fdir1>
       <material>Gazebo/Grey</material>
     </gazebo>

File: ranger/ranger_mini/urdf/ranger_mini.urdf (robot description, URDF)
Before this commit: robot ranger_mini, 9 links, 8 joints
Links:
- removed link ffr_wheel_ink
- added link ffr_wheel_link, mass 1.1364; collision mesh filename=package://ranger_mini/meshes/ffr_wheel_link.STL; visual mesh filename=package://ranger_mini/meshes/ffr_wheel_link.STL
Joints:
- removed joint fron_left_steering_joint
- added joint front_left_steering_joint: type continuous, parent base_link, child front_left_steering_link, origin xyz=0.26366 0.18001 0.0557 rpy=3.1416 0 1.5708, axis 0 0 1
- joint ffr_wheel_joint: child ffr_wheel_ink -> ffr_wheel_link
- joint rfl_wheel_joint: axis -1 0 0 -> 1 0 0

File: ranger/ranger_mini/urdf/ranger_mini.xacro (robot description, xacro)
@@ -4,5 +4,4 @@
      For more information, please see http://wiki.ros.org/sw_urdf_exporter -->
 <robot name="ranger_mini" xmlns:xacro="http://ros.org/wiki/xacro">
-  <xacro:include filename="$(find ranger_mini)/urdf/ranger_mini.gazebo.xacro"/>
   <link
     name="base_link">
@@ -98,4 +97,5 @@
       xyz="0 0 1" />
     <limit effort="5" velocity="6.28"  lower="-2.1" upper="2.1" />
+    <dynamics damping="0.0" friction="5"/>
   </joint>
   <link
@@ -152,4 +152,5 @@
       xyz="1 0 0" />
     <limit effort="1.5" velocity="20"/>
+    <dynamics damping="0.0" friction="2"/>
   </joint>
   <link
@@ -206,4 +207,5 @@
       xyz="0 0 1" />
     <limit effort="5" velocity="6.28"  lower="-2.1" upper="2.1" />
+       <dynamics damping="0.0" friction="5"/>
   </joint>
   <link
@@ -260,4 +262,5 @@
       xyz="1 0 0" />
     <limit effort="1.5" velocity="20"/>
+        <dynamics damping="0.0" friction="2"/>
   </joint>
   <link
@@ -314,4 +317,5 @@
       xyz="0 0 1" />
     <limit effort="5" velocity="6.28"  lower="-2.1" upper="2.1" />
+        <dynamics damping="0.0" friction="5"/>
   </joint>
   <link
@@ -368,4 +372,5 @@
       xyz="1 0 0" />
     <limit effort="1.5" velocity="20"/>
+        <dynamics damping="0.0" friction="2"/>
   </joint>
   <link
@@ -422,4 +427,5 @@
       xyz="0 0 1" />
     <limit effort="5" velocity="6.28"  lower="-2.1" upper="2.1" />
+        <dynamics damping="0.0" friction="5"/>
   </joint>
   <link
@@ -476,5 +482,7 @@
       xyz="1 0 0" />
       <limit effort="1.5" velocity="20"/>
-  </joint>
+          <dynamics damping="0.0" friction="2"/>
+  </joint>
+  <xacro:include filename="$(find ranger_mini)/urdf/ranger_mini.gazebo.xacro"/>
 	<transmission name="front_left_steering_trans">
       <type>transmission_interface/SimpleTransmission</type>

File: ranger/ranger_mini_gazebo/xacro/ranger_mini.gazebo.xacro (robot description, xacro)
@@ -35,24 +35,44 @@
     <gazebo reference="ffl_wheel_link">
       <!-- <selfCollide>false</selfCollide> -->
-      <mu1 value="10" />
-      <mu2 value="10" />
+    <mu1>0.8</mu1>
+    <mu2>0.8</mu2>
+    <kp>10000000.0</kp>
+    <kd>1.0</kd>
+    <minDepth>0.001</minDepth>
+    <maxVel>0.1</maxVel>
+    <fdir1>1 0 0</fdir1>
       <material>Gazebo/Grey</material>
     </gazebo>
     <gazebo reference="ffr_wheel_link">
       <!-- <selfCollide>false</selfCollide> -->
-      <mu1 value="10" />
-      <mu2 value="10" />
+      <mu1>0.8</mu1>
+    <mu2>0.8</mu2>
+    <kp>10000000.0</kp>
+    <kd>1.0</kd>
+    <minDepth>0.001</minDepth>
+    <maxVel>0.1</maxVel>
+    <fdir1>1 0 0</fdir1>
       <material>Gazebo/Grey</material>
     </gazebo>
     <gazebo reference="rfl_wheel_link">
       <!-- <selfCollide>false</selfCollide> -->
-      <mu1 value="10" />
-      <mu2 value="10" />
+      <mu1>0.8</mu1>
+    <mu2>0.8</mu2>
+    <kp>10000000.0</kp>
+    <kd>1.0</kd>
+    <minDepth>0.001</minDepth>
+    <maxVel>0.1</maxVel>
+    <fdir1>1 0 0</fdir1>
       <material>Gazebo/Grey</material>
     </gazebo>
     <gazebo reference="rfr_wheel_link">
       <!-- <selfCollide>false</selfCollide> -->
-      <mu1 value="10" />
-      <mu2 value="10" />
+      <mu1>0.8</mu1>
+    <mu2>0.8</mu2>
+    <kp>10000000.0</kp>
+    <kd>1.0</kd>
+    <minDepth>0.001</minDepth>
+    <maxVel>0.1</maxVel>
+    <fdir1>1 0 0</fdir1>
       <material>Gazebo/Grey</material>
     </gazebo>
