Commit message: update modle and fix bug

File: ranger/ranger_mini/urdf/ranger_mini_gazebo.xacro (robot description, xacro)
@@ -82,4 +82,5 @@
             <child link="fl_wheel_link"/>
             <axis xyz="0 1 0" rpy="0 0 0" />
+            <limit effort="100" velocity="10" />
         </joint>
    <link name="fr_steering_wheel_link">
@@ -138,4 +139,5 @@
             <child link="fr_wheel_link"/>
             <axis xyz="0 1 0" rpy="0 0 0" />
+            <limit effort="100" velocity="10" />
         </joint>
    <link name="rl_steering_wheel_link">
@@ -194,4 +196,5 @@
             <child link="rl_wheel_link"/>
             <axis xyz="0 1 0" rpy="0 0 0" />
+            <limit effort="100" velocity="10" />
         </joint>
    <link name="rr_steering_wheel_link">
@@ -250,4 +253,5 @@
             <child link="rr_wheel_link"/>
             <axis xyz="0 1 0" rpy="0 0 0" />
+            <limit effort="100" velocity="10" />
         </joint>
 	<transmission name="fl_steering_wheel_trans">
@@ -342,4 +346,5 @@
       <state_interface name="velocity"/>
       <state_interface name="effort"/>
+      <state_interface name="position"/>
     </joint>
     <joint name="fr_wheel">
@@ -350,4 +355,5 @@
       <state_interface name="velocity"/>
       <state_interface name="effort"/>
+      <state_interface name="position"/>
     </joint>
     <joint name="rl_wheel">
@@ -358,4 +364,5 @@
       <state_interface name="velocity"/>
       <state_interface name="effort"/>
+      <state_interface name="position"/>
     </joint>
     <joint name="rr_wheel">
@@ -366,4 +373,5 @@
       <state_interface name="velocity"/>
       <state_interface name="effort"/>
+      <state_interface name="position"/>
     </joint>
     <joint name="fl_steering_wheel">
@@ -404,23 +412,7 @@
     </joint>
   </ros2_control>
-<!-- <gazebo>
-    <plugin name="object_controller" filename="libgazebo_ros_planar_move.so">
-      <ros>
-        <namespace>/</namespace>
-      </ros>
-      <update_rate>100</update_rate>
-      <publish_rate>10</publish_rate>
-      <publish_odom>true</publish_odom>
-      <publish_odom_tf>true</publish_odom_tf>
-      <odometry_frame>demo</odometry_frame>
-      <robot_base_frame>link</robot_base_frame>
-      <covariance_x>0.0001</covariance_x>
-      <covariance_y>0.0001</covariance_y>
-      <covariance_yaw>0.01</covariance_yaw>
-    </plugin>
-</gazebo> -->
     <gazebo>
         <plugin name="gazebo_ros2_control" filename="libgazebo_ros2_control.so">
-            <parameters>/home/agilex/ugv_sim/src/ranger_mini/config/ranger_mini_joint.yaml</parameters>
+            <parameters>/home/agilex/ugv_sim_ws/src/ugv_gazebo_sim/ranger/ranger_mini/config/ranger_mini_joint.yaml</parameters>
         </plugin>
     </gazebo>
