Commit message: add lidar to scout_mini

File: scout/scout_description/urdf/mini.xacro (robot description, xacro)
@@ -8,4 +8,6 @@
     <xacro:include filename="$(find scout_description)/urdf/scout_mini_wheel_3.xacro" />
     <xacro:include filename="$(find scout_description)/urdf/scout_mini_wheel_4.xacro" />
+    <xacro:include filename="$(find scout_description)/urdf/scout_mini_lidar.xacro" />
+    <xacro:include filename="$(find scout_description)/urdf/inertial_macros.xacro"/>
     <!-- Variables -->
     <xacro:property name="M_PI" value="3.14159"/>
@@ -17,4 +19,8 @@
     <xacro:property name="track" value="0.416503"/>
     <xacro:property name="wheel_vertical_offset" value="-0.100998" />
+    <!-- Colors -->
+    <material name="black">
+        <color rgba="0.0 0.0 0.0 1"/>
+    </material>
 <!--    <xacro:property name="track" value="0.3426" />
     <xacro:property name="wheelbase" value="0.3181"/>

File: scout/scout_description/urdf/scout_mini.xacro (robot description, xacro)
@@ -8,4 +8,5 @@
     <xacro:include filename="$(find scout_description)/urdf/scout_mini_wheel_3.xacro" />
     <xacro:include filename="$(find scout_description)/urdf/scout_mini_wheel_4.xacro" />
+    <xacro:include filename="scout_mini_lidar.xacro"/>
     <!-- Variables -->
     <xacro:property name="M_PI" value="3.14159"/>

Commit message: adding SLAM and NAV2 support

File: scout/scout_description/urdf/mini.xacro (robot description, xacro)
@@ -47,4 +47,12 @@
           </geometry>
         </collision>
+    </link>
+    <!-- BASE_FOOTPRINT LINK -->
+    <joint name="base_footprint_joint" type="fixed">
+        <parent link="base_link"/>
+        <child link="base_footprint"/>
+        <origin xyz="0 0 0" rpy="0 0 0"/>
+    </joint>
+    <link name="base_footprint">
     </link>
     <!-- <joint name="chassis_link_joint" type="fixed">
