Commit message: add ranger_mini.urdf and repair ranger_mini_gazebo.xacro

File: ranger_mini/ranger_mini_v3_gazebo/xacro/ranger_mini_gazebo.xacro (robot description, xacro)
@@ -100,5 +100,5 @@
             </visual>
             <collision>
-                <origin xyz="0 0 0" rpy="1.57 0 0" />
+                <origin xyz="0 0 -0.005" rpy="1.57 0 0" />
                 <geometry>
                     <cylinder length="0.08" radius="0.09" />
@@ -270,5 +270,5 @@
             </visual>
             <collision>
-                <origin xyz="0 0 0" rpy="1.57 0 0" />
+                <origin xyz="0.005 0.005 -0.005" rpy="1.57 0 0" />
                 <geometry>
                     <cylinder length="0.08" radius="0.09" />
@@ -326,5 +326,5 @@
             </visual>
             <collision>
-                <origin xyz="0 0 0" rpy="1.57 0 0" />
+                <origin xyz="-0.015 0.02 -0.005" rpy="1.57 0 0" />
                 <geometry>
                     <cylinder length="0.08" radius="0.09" />

Commit message: 解决ranger_mini v3 抖动的问题

File: ranger_mini/ranger_mini_v3_gazebo/xacro/ranger_mini_gazebo.xacro (robot description, xacro)
@@ -84,5 +84,5 @@
     <axis
       xyz="0 0 -1" />
-    <limit effort="5" velocity="6.28"  lower="-2.1" upper="2.1" />
+    <limit effort="5" velocity="1"  lower="-2.1" upper="2.1" />
   </joint>
         <link name="fr_wheel_link">
@@ -168,5 +168,5 @@
     <axis
       xyz="0 0 -1" />
-        <limit effort="5" velocity="6.28"  lower="-2.1" upper="2.1" />
+        <limit effort="5" velocity="1"  lower="-2.1" upper="2.1" />
   </joint>
         <link name="fl_wheel_link">
@@ -252,5 +252,5 @@
     <axis
       xyz="0 0 -1" />
-        <limit effort="5" velocity="6.28"  lower="-2.1" upper="2.1" />
+        <limit effort="5" velocity="1"  lower="-2.1" upper="2.1" />
   </joint>
         <link name="rl_wheel_link">
@@ -308,5 +308,5 @@
         <child link="rr_steering_wheel_link"/>
         <axis xyz="0 0 -1" rpy="0 0 0" />
-        <limit effort="5" velocity="6.28"  lower="-2.1" upper="2.1" />
+        <limit effort="5" velocity="1"  lower="-2.1" upper="2.1" />
     </joint>
        <link name="rr_wheel_link">
