Commit message: 修复ranger_air urdf模型

File: ranger_air/ranger_air_description/urdf/ranger_air_description.urdf (robot description, URDF)
Before this commit: robot ranger_air_description, 13 links, 12 joints
Links:
- link camera_link: geometry collision mesh filename=package://ranger_air_description/meshes/dae/camera_link.dae; visual mesh filename=package://ranger_air_description/meshes/dae/camera_link.dae
- link fl_steering_link: geometry collision mesh filename=package://ranger_air_description/meshes/dae/fl_streering_li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; visual mesh filename=package://ranger_air_description/meshes/dae/fl_streering_li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
- link fl_wheel_link: geometry collision mesh filename=package://ranger_air_description/meshes/dae/fl_wheel_link.d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; visual mesh filename=package://ranger_air_description/meshes/dae/fl_wheel_link.d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
- link fr_steering_link: geometry collision mesh filename=package://ranger_air_description/meshes/dae/fr_steering_lin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; visual mesh filename=package://ranger_air_description/meshes/dae/fr_steering_lin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
- link fr_wheel_link: geometry collision mesh filename=package://ranger_air_description/meshes/dae/fr_wheel_link.d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; visual mesh filename=package://ranger_air_description/meshes/dae/fr_wheel_link.d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
- link rl_steering_link: geometry collision mesh filename=package://ranger_air_description/meshes/dae/rl_steering_lin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; visual mesh filename=package://ranger_air_description/meshes/dae/rl_steering_lin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
- link rl_wheel_link: geometry collision mesh filename=package://ranger_air_description/meshes/dae/rl_wheel_link.d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; visual mesh filename=package://ranger_air_description/meshes/dae/rl_wheel_link.d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
- link rr_steering_link: geometry collision mesh filename=package://ranger_air_description/meshes/dae/rr_steering_lin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; visual mesh filename=package://ranger_air_description/meshes/dae/rr_steering_lin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
- link rr_wheel_link: geometry collision mesh filename=package://ranger_air_description/meshes/dae/rr_wheel_link.d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; visual mesh filename=package://ranger_air_description/meshes/dae/rr_wheel_link.d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
