Commit message: add ranger_air and ranger_delta；fixed hunter se bug

File: hunter_se/hunter_se_gazebo/xacro/hunter_se_gazebo.xacro (robot description, xacro)
@@ -54,10 +54,10 @@
         value="0.5" />
       <inertia
-        ixx="0.0222"
+        ixx="0.000222"
         ixy="0.0"
         ixz="0.0"
-        iyy="0.0222"
+        iyy="0.000222"
         iyz="0.0"
-        izz="0.0378075" />
+        izz="0.000378075" />
     </inertial>
     <visual>
@@ -85,5 +85,5 @@
   <joint
     name="fr_steer_left_joint"
-    type="continuous">
+    type="revolute">
     <origin
       xyz="0.34058 0.24619 -0.1535"
@@ -96,6 +96,6 @@
       xyz="0 0 1" />
     <limit
-      lower="-0.69"
-      upper="0.69"
+      lower="-0.52"
+      upper="0.52"
       effort="10"
       velocity="0.69" />
@@ -108,12 +108,12 @@
         rpy="0 0 0" />
       <mass
-        value="1" />
-      <inertia
-        ixx="0.0222"
+        value="3" />
+      <inertia
+        ixx="0.014583"
         ixy="0.0"
         ixz="0.0"
-        iyy="0.0222"
+        iyy="0.014583"
         iyz="0.0"
-        izz="0.0378075" />
+        izz="0.0281535"/>
     </inertial>
     <visual>
@@ -138,5 +138,5 @@
         <!-- <mesh
           filename="file://$(find hunter_se_description)/meshes/fr_left_link.STL" /> -->
-          <cylinder radius="0.13" length="0.045"/>
+          <cylinder radius="0.137" length="0.045"/>
       </geometry>
     </collision>
@@ -154,5 +154,5 @@
     <axis
       xyz="0 0 -1" />
-    <limit effort="10" velocity="100" />
+    <limit effort="10" velocity="1" />
   </joint>
   <link
@@ -163,12 +163,12 @@
         rpy="0 0 0" />
       <mass
-        value="1" />
-      <inertia
-        ixx="0.0222"
+        value="0.5" />
+      <inertia
+        ixx="0.000222"
         ixy="0.0"
         ixz="0.0"
-        iyy="0.0222"
+        iyy="0.000222"
         iyz="0.0"
-        izz="0.0378075" />
+        izz="0.000378075" />
     </inertial>
     <visual>
@@ -196,5 +196,5 @@
   <joint
     name="fr_steer_right_joint"
-    type="continuous">
+    type="revolute">
     <origin
       xyz="0.34219 -0.24619 -0.1535"
@@ -207,6 +207,6 @@
       xyz="0 0 1" />
     <limit
-      lower="-0.69"
-      upper="0.69"
+      lower="-0.52"
+      upper="0.52"
       effort="10"
       velocity="0.69" />
@@ -219,12 +219,12 @@
         rpy="0 0 0" />
       <mass
-        value="1" />
-      <inertia
-        ixx="0.0222"
+        value="3" />
+      <inertia
+        ixx="0.014583"
         ixy="0.0"
         ixz="0.0"
-        iyy="0.0222"
+        iyy="0.014583"
         iyz="0.0"
-        izz="0.0378075" />
+        izz="0.0281535"/>
     </inertial>
     <visual>
@@ -249,5 +249,5 @@
         <!-- <mesh
           filename="file://$(find hunter_se_description)/meshes/fr_right_link.STL" /> -->
-          <cylinder radius="0.13" length="0.045"/>
+          <cylinder radius="0.137" length="0.045"/>
       </geometry>
     </collision>
@@ -265,5 +265,5 @@
     <axis
       xyz="0 0 1" />
-    <limit effort="10" velocity="100" />
+    <limit effort="10" velocity="1" />
   </joint>
   <link
@@ -274,12 +274,12 @@
         rpy="0 0 0" />
       <mass
-        value="1" />
-      <inertia
-        ixx="0.0222"
+        value="3" />
+      <inertia
+        ixx="0.014583"
         ixy="0.0"
         ixz="0.0"
-        iyy="0.0222"
+        iyy="0.014583"
         iyz="0.0"
-        izz="0.0378075" />
+        izz="0.0281535"/>
     </inertial>
     <visual>
@@ -304,5 +304,5 @@
         <!-- <mesh
           filename="file://$(find hunter_se_description)/meshes/re_left_link.STL" /> -->
-          <cylinder radius="0.13" length="0.045"/>
+          <cylinder radius="0.137" length="0.045"/>
       </geometry>
     </collision>
@@ -320,5 +320,5 @@
     <axis
       xyz="0 0 -1" />
-    <limit effort="10" velocity="100" />
+    <limit effort="10" velocity="1" />
   </joint>
   <link
@@ -329,12 +329,12 @@
         rpy="0 0 0" />
       <mass
-        value="1" />
-      <inertia
-        ixx="0.0222"
+        value="3" />
+      <inertia
+        ixx="0.014583"
         ixy="0.0"
         ixz="0.0"
-        iyy="0.0222"
+        iyy="0.014583"
         iyz="0.0"
-        izz="0.0378075" />
+        izz="0.0281535"/>
     </inertial>
     <visual>
@@ -359,5 +359,5 @@
         <!-- <mesh
           filename="file://$(find hunter_se_description)/meshes/re_right_link.STL" /> -->
-          <cylinder radius="0.13" length="0.045"/>
+          <cylinder radius="0.137" length="0.045"/>
       </geometry>
     </collision>
@@ -375,5 +375,5 @@
     <axis
       xyz="0 0 1" />
-    <limit effort="10" velocity="100" />
+    <limit effort="10" velocity="1" />
   </joint>
   <link
